Commit message: 20251103

File: omorobot_description/urdf/DONKEYBOTI.urdf (robot description, URDF)
Before this commit: robot DONKEYBOTI, 6 links, 5 joints
Links:
- link base_scan: geometry visual mesh filename=package://omorobot_description/meshes/sensors/TMINIPRO.stl scale=0.001 0.001 0.001

File: omorobot_description/urdf/R2MINI.urdf (robot description, URDF)
Before this commit: robot R2MINI, 6 links, 5 joints
Links:
- removed link imu_link
- link base_link: geometry collision box size=0.2 0.19 0.16; visual mesh filename=package://omorobot_description/meshes/bases/R2MINI_BODY.stl scale=0.001 0.001 0.001
- link base_scan: geometry collision cylinder length=0.012 radius=0.019; visual cylinder length=0.012 radius=0.019
- link wheel_left_link: geometry collision cylinder length=0.027 radius=0.034; visual mesh filename=package://omorobot_description/meshes/wheels/R2MINI_WHEEL.s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 scale=0.001 0.001 0.001
- link wheel_right_link: geometry collision cylinder length=0.027 radius=0.034; visual mesh filename=package://omorobot_description/meshes/wheels/R2MINI_WHEEL.s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 scale=0.001 0.001 0.001
Joints:
- removed joint imu_joint
- joint base_joint: origin xyz=0.0 0.0 0.016 rpy=0.0 0.0 0.0 -> xyz=0.0 0.0 0.018 rpy=0.0 0.0 0.0
- joint scan_joint: origin xyz=0.01 0.0 0.149 rpy=0.0 0.0 0.0 -> xyz=0.0155 0.0 0.064 rpy=3.14 0.0 0.0
- joint wheel_left_joint: origin xyz=0.0 0.09 0.02 rpy=-1.57 0.0 0.0 -> xyz=0.0 0.09 0.015 rpy=-1.57 0.0 0.0
- joint wheel_right_joint: origin xyz=0.0 -0.09 0.02 rpy=-1.57 0.0 0.0 -> xyz=0.0 -0.09 0.015 rpy=-1.57 0.0 0.0
